Commit message: Added camera and markers

File: tortoisebotpromax_description/urdf/tortoisebotpromax.xacro (robot description, xacro)
@@ -5,4 +5,9 @@
 <xacro:include filename="$(find tortoisebotpromax_description)/gazebo/tortoisebotpromax_materials.gazebo" />
 <xacro:include filename="$(find tortoisebotpromax_description)/gazebo/tortoisebotpromax_physics.gazebo" />
+<!-- <xacro:include filename="$(find realsense_ros_gazebo)/xacro/depthcam.xacro"/> -->
+<xacro:include filename="$(find realsense2_description)/urdf/_d435.urdf.xacro" />
+<!-- <xacro:realsense_d435 sensor_name="ttbpromax" parent_link="realsense_1" rate="10">
+  <origin xyz="0.011753067204287801 -0.0004295385558066378 -0.035091351352319555" rpy="0 0 0"/>
+</xacro:realsense_d435> -->
 <link name="base_link">
   <inertial>
@@ -25,6 +30,9 @@
   </collision>
 </link>
+<xacro:sensor_d435 name="camera" topics_ns="camera" parent="realsense_1" publish_pointcloud="true">
+  <origin xyz="0.011753067204287801 -0.0004295385558066378 -0.035091351352319555" rpy="0 0 0"/>
+</xacro:sensor_d435>
 <link name="realsense_1">
-  <inertial>
+  <!-- <inertial>
     <origin xyz="0.011753067204287801 -0.0004295385558066378 -0.035091351352319555" rpy="0 0 0"/>
     <mass value="0.34623874488058043"/>
@@ -43,5 +51,5 @@
       <mesh filename="package://tortoisebotpromax_description/meshes/realsense_1.stl" scale="0.001 0.001 0.001"/>
     </geometry>
-  </collision>
+  </collision> -->
 </link>
 <link name="right_wheel_1">

Commit message: updated with new world

File: tortoisebotpromax_description/urdf/tortoisebotpromax.xacro (robot description, xacro)
@@ -5,9 +5,9 @@
 <xacro:include filename="$(find tortoisebotpromax_description)/gazebo/tortoisebotpromax_materials.gazebo" />
 <xacro:include filename="$(find tortoisebotpromax_description)/gazebo/tortoisebotpromax_physics.gazebo" />
-<!-- <xacro:include filename="$(find realsense_ros_gazebo)/xacro/depthcam.xacro"/> -->
+<!-- Realsense xacro -->
 <xacro:include filename="$(find realsense2_description)/urdf/_d435.urdf.xacro" />
-<!-- <xacro:realsense_d435 sensor_name="ttbpromax" parent_link="realsense_1" rate="10">
-  <origin xyz="0.011753067204287801 -0.0004295385558066378 -0.035091351352319555" rpy="0 0 0"/>
-</xacro:realsense_d435> -->
+<material name="silver">
+  <color rgba="0.700 0.700 0.700 1.000"/>
+</material>
 <link name="base_link">
   <inertial>
@@ -30,4 +30,5 @@
   </collision>
 </link>
+<!-- Realsense Plugin  -->
 <xacro:sensor_d435 name="camera" topics_ns="camera" parent="realsense_1" publish_pointcloud="true">
   <origin xyz="0.011753067204287801 -0.0004295385558066378 -0.035091351352319555" rpy="0 0 0"/>

Commit message: realsense dependencies fix

File: tortoisebotpromax_description/urdf/tortoisebotpromax.xacro (robot description, xacro)
@@ -5,9 +5,9 @@
 <xacro:include filename="$(find tortoisebotpromax_description)/gazebo/tortoisebotpromax_materials.gazebo" />
 <xacro:include filename="$(find tortoisebotpromax_description)/gazebo/tortoisebotpromax_physics.gazebo" />
-<!-- Realsense xacro -->
+<!-- <xacro:include filename="$(find realsense_ros_gazebo)/xacro/depthcam.xacro"/> -->
 <xacro:include filename="$(find realsense2_description)/urdf/_d435.urdf.xacro" />
-<material name="silver">
-  <color rgba="0.700 0.700 0.700 1.000"/>
-</material>
+<!-- <xacro:realsense_d435 sensor_name="ttbpromax" parent_link="realsense_1" rate="10">
+  <origin xyz="0.011753067204287801 -0.0004295385558066378 -0.035091351352319555" rpy="0 0 0"/>
+</xacro:realsense_d435> -->
 <link name="base_link">
   <inertial>
@@ -30,5 +30,4 @@
   </collision>
 </link>
-<!-- Realsense Plugin  -->
 <xacro:sensor_d435 name="camera" topics_ns="camera" parent="realsense_1" publish_pointcloud="true">
   <origin xyz="0.011753067204287801 -0.0004295385558066378 -0.035091351352319555" rpy="0 0 0"/>
